File: hardware/boards/glasgow/io_buffer.sch (KiCad schematic (older format))
At the start: 21 parts, among them J2 Conn_02x10_Odd_Even, U10 DAC081C081CIMK, U11 TPS73101DBV, U5 FXMA108BQX, U9 ADC081C021CIMM

Commit message: Initial Rev C IO cell schematic.
Parts:
- removed RN3: R_Pack08, Resistor_SMD:R_Array_Convex_8x0602, symbol Device:R_Pack08
- removed U5: FXMA108BQX, Package_DFN_QFN:WQFN-20-1EP_2.5x4.5mm_P0.5mm_EP1x2.9mm, symbol Logic_LevelTranslator:FXMA108
- added C32, C47, C48, C49, C50, C51, C52, C53, C54, C55, C56, C57, C58, C59: u1, Capacitor_SMD:C_0603_1608Metric_Pad0.99x1.00mm_HandSolder, symbol Device:C
- added RN2: R_Pack08, Resistor_SMD:R_Array_Convex_8x0602, symbol Device:R_Pack08
- added U16, U17, U18, U19, U20, U21, U5, U6: SN74LVC1T45DRL, Package_TO_SOT_SMD:SOT-563, symbol Logic_LevelTranslator:SN74LVC1T45DRL
Connections:
- net labels added: DIR0, DIR1, DIR2, DIR3, DIR4, DIR5, DIR6, DIR7, VEXT
- net labels removed: X0, X1, X2, X3, X4, X5, X6, X7, ~OE
- wire segments 140 -> 193
Other:
- note added: "Imax @ 3V3 = 32 mA each\nImax @ Vtg = 32 mA each"
- note added: "LDO Input Cap"
- note removed: "Imax @ 3V3 = 35 mA\nImax @ Vtg = 35 mA"
- moved on the sheet: U11
