File: hardware/boards/glasgow/glasgow.sch (KiCad schematic (older format))
At the start: 77 parts, among them J1 USB_B_Micro, J4 Conn_01x02, U1 CY7C68013A-56LTX, U15 TPD3S014, U2 CAT24M01W, U3 CAT24C256W, U4 ICE40UP5K-SG48ITR, U7 LM3880MF-1AF, U8 MIC5355-S4YMME, Y1 24M

Commit message: Refactor FX2 into hierarchical subsheet.
Parts:
- removed C1: 4u7, Capacitor_SMD:C_0603_1608Metric_Pad0.99x1.00mm_HandSolder, symbol Device:C
- removed C10, C2, C3, C4, C5, C6, C7, C9: u1, Capacitor_SMD:C_0603_1608Metric_Pad0.99x1.00mm_HandSolder, symbol Device:C
- removed C11, C12: 18p, Capacitor_SMD:C_0603_1608Metric_Pad0.99x1.00mm_HandSolder, symbol Device:C
- removed R11, R17, R18, R19, R4, R9: 100k, Resistor_SMD:R_0603_1608Metric_Pad0.99x1.00mm_HandSolder, symbol Device:R
- removed TP6: CLKREF, TestPoint:TestPoint_Pad_D1.0mm, symbol Connector:Test_Point
- removed TP7: 3V3, TestPoint:TestPoint_Pad_D1.0mm, symbol Connector:Test_Point
- removed U1: CY7C68013A-56LTX, Package_DFN_QFN:Cypress_QFN-56-1EP_8x8mm_P0.5mm_EP6.22x6.22mm_ThermalVias, symbol MCU_Cypress:CY7C68013A-56LTX
- removed Y1: 24M, Crystals:Crystal_SMD_3225-4pin_3.2x2.5mm, symbol Device:Crystal_GND24
Connections:
- net labels removed: FPGA_DONE, XTALIN, XTALOUT
- wire segments 393 -> 262
Other:
- note removed: "Alternate use for\nFLAGD pin: INT1"
- note removed: "FPGA reset asserted\non tristate"
- note removed: "Imax(USB) @ 3V3 = 80 mA\nImax @ 3V3 = 209 mA"
